File: test1.kicad_sch (KiCad schematic)
At the start: 0 parts

Commit message: first changed
Other:
- sheet 3 renamed RJ45
- added sheet POWER (POWER.kicad_sch)
- sheet RJ45: file untitled.kicad_sch -> 2.5g-Eethrnet.kicad_sch
